Commit message: 실물 robot.launch.xml 이 WeGo URDF·카메라 static TF 3 개 대신 우리 URDF 하나로 TF 를 내게: 카메라를 orbbec_dabai.xacro 모듈로 빼고 장착 위치를 실측 (0.15, −0.005, 0.06) 으로, color·depth 프레임은 드라이버만 냄

File: src/limo_fire/limo_fire_description/urdf/limo_fire.urdf.xacro (robot description, xacro)
@@ -1,6 +1,17 @@
 <?xml version="1.0"?>
-<!-- 화재 대응 LIMO Pro. 지금은 기본 몸체만. 열화상·레이더·초음파·노즐(팬·틸트)은 배치가 정해지면 모듈 xacro 로 더한다. -->
+<!-- 화재 대응 LIMO Pro 조립. 모듈마다 xacro 하나, 장착 위치는 여기 한 곳에만 둔다.
+     열화상·레이더·초음파·노즐(팬·틸트)은 배치가 정해지면 모듈 xacro 를 더하고 여기서 부른다.
+     xacro limo_fire.urdf.xacro camera_pitch:=0.0 camera_driver_tf:=false -->
 <robot name="limo_fire" xmlns:xacro="http://ros.org/wiki/xacro">
+  <!-- 카메라 마운트 틸트(라디안, 아래로 숙이면 +). 손으로 고정하는 마운트라 관절이 아니라 인자로 받는다 -->
+  <xacro:arg name="camera_pitch" default="0.0"/>
+  <!-- true: 실물 — camera_link 아래 color·depth 프레임은 Orbbec 드라이버가 낸다 -->
+  <xacro:arg name="camera_driver_tf" default="false"/>
   <xacro:include filename="$(find limo_fire_description)/urdf/limo_pro_base.xacro"/>
+  <xacro:include filename="$(find limo_fire_description)/urdf/orbbec_dabai.xacro"/>
   <xacro:limo_pro_base/>
+  <!-- base_link → camera_link. x·y 는 실물 실측(약 0.15, −0.005), z 는 WeGo 틸트 TF 값 그대로(실측 필요).
+       이전 값: WeGo static TF (0.23, 0.05, 0.06), Webots (0.096, 0.015, 0.03) -->
+  <xacro:orbbec_dabai parent="base_link" name="camera" xyz="0.15 -0.005 0.06"
+                      pitch="$(arg camera_pitch)" driver_tf="$(arg camera_driver_tf)"/>
 </robot>

File: src/limo_fire/limo_fire_description/urdf/limo_pro_base.xacro (robot description, xacro)
@@ -1,7 +1,5 @@
 <?xml version="1.0"?>
-<!-- LIMO Pro 기본 몸체: 바퀴 4 개(차동) + 라이다 + IMU + depth 카메라.
+<!-- LIMO Pro 기본 몸체: 바퀴 4 개(차동) + 라이다 + IMU. 카메라는 orbbec_dabai.xacro, 장착 위치는 limo_fire.urdf.xacro.
      몸통·바퀴·라이다·IMU 는 WeGo limo_description 의 limo_four_diff.xacro 와 같은 값(매크로도 그것을 씀).
-     카메라는 WeGo 차동 모델에 없어서, 교수님 Webots 환경(webots_ros2_limo robot_launch.py)이 실제 몸통 메시의
-     카메라 자리에 맞춘 값을 쓴다: base_link → camera_link (0.096, 0.015, 0.03).
      base_link 는 바닥에서 0.145 m (바퀴 중심 -0.10 + 바퀴 반지름 0.045). base_footprint 는 두지 않는다(실물 드라이버에 없음). -->
 <robot xmlns:xacro="http://ros.org/wiki/xacro">
@@ -17,12 +15,4 @@
   <xacro:property name="wheel_length" value="0.045" />
   <xacro:property name="wheel_radius" value="0.045" />
-  <xacro:macro name="optical_frame" params="parent name">
-    <link name="${name}_optical_frame"/>
-    <joint name="${name}_optical_joint" type="fixed">
-      <origin xyz="0 0 0" rpy="${-M_PI/2} 0 ${-M_PI/2}"/>
-      <parent link="${parent}"/>
-      <child link="${name}_optical_frame"/>
-    </joint>
-  </xacro:macro>
   <xacro:macro name="limo_pro_base">
     <link name="base_link">
@@ -66,25 +56,4 @@
       <origin xyz="${-wheelbase/2} ${-track/2} ${wheel_vertical_offset}" rpy="${M_PI} 0 0" />
     </xacro:limo_wheel>
-    <!-- depth 카메라(Orbbec): camera_link 장착 + color·depth 흐름 프레임(Orbbec 드라이버와 같은 이름) + 광학 프레임(z 앞) -->
-    <link name="camera_link"/>
-    <joint name="camera_joint" type="fixed">
-      <origin xyz="0.096 0.015 0.03" rpy="0 0 0"/>
-      <parent link="base_link"/>
-      <child link="camera_link"/>
-    </joint>
-    <link name="camera_color_frame"/>
-    <joint name="camera_color_joint" type="fixed">
-      <origin xyz="0.00015 -0.03 0.00002" rpy="0 0 0"/>
-      <parent link="camera_link"/>
-      <child link="camera_color_frame"/>
-    </joint>
-    <xacro:optical_frame parent="camera_color_frame" name="camera_color"/>
-    <link name="camera_depth_frame"/>
-    <joint name="camera_depth_joint" type="fixed">
-      <origin xyz="0 0 0" rpy="0 0 0"/>
-      <parent link="camera_link"/>
-      <child link="camera_depth_frame"/>
-    </joint>
-    <xacro:optical_frame parent="camera_depth_frame" name="camera_depth"/>
   </xacro:macro>
 </robot>

Commit message: Webots 시뮬 맵 3 개(덕트호스 미로·사무실·창고)에 YOLO 7 클래스 물체를 놓고, sim.launch.xml world:=<맵> 하나로 실물과 같은 지도·Nav2·인식 launch 를 띄우는 구조(sim_robot.launch.xml·공용 URDF description.launch.xml·launch 인자 공용화), Nav2 팽창 반경 0.45 m·yolo mapper 조건 수정, 4 맵 시뮬 지도 + 순찰 전부 도착

File: src/limo_fire/limo_fire_description/urdf/limo_fire.urdf.xacro (robot description, xacro)
@@ -2,16 +2,20 @@
 <!-- 화재 대응 LIMO Pro 조립. 모듈마다 xacro 하나, 장착 위치는 여기 한 곳에만 둔다.
      열화상·레이더·초음파·노즐(팬·틸트)은 배치가 정해지면 모듈 xacro 를 더하고 여기서 부른다.
-     xacro limo_fire.urdf.xacro camera_pitch:=0.0 camera_driver_tf:=false -->
+     xacro limo_fire.urdf.xacro platform:=real camera_pitch:=0.0 camera_driver_tf:=false -->
 <robot name="limo_fire" xmlns:xacro="http://ros.org/wiki/xacro">
+  <!-- real: 실물 LIMO, webots: 교수님 Webots 모델(webots_ros2_limo LimoFourDiff.proto). 둘이 다른 장착 위치만 여기서 고른다 -->
+  <xacro:arg name="platform" default="real"/>
   <!-- 카메라 마운트 틸트(라디안, 아래로 숙이면 +). 손으로 고정하는 마운트라 관절이 아니라 인자로 받는다 -->
   <xacro:arg name="camera_pitch" default="0.0"/>
-  <!-- true: 실물 — camera_link 아래 color·depth 프레임은 Orbbec 드라이버가 낸다 -->
+  <!-- true: camera_link 아래 color·depth 프레임은 카메라 드라이버가 낸다 (실물 Orbbec 드라이버, Webots limo_sensors 플러그인 둘 다) -->
   <xacro:arg name="camera_driver_tf" default="false"/>
   <xacro:include filename="$(find limo_fire_description)/urdf/limo_pro_base.xacro"/>
   <xacro:include filename="$(find limo_fire_description)/urdf/orbbec_dabai.xacro"/>
   <xacro:limo_pro_base/>
-  <!-- base_link → camera_link. x·y 는 실물 실측(약 0.15, −0.005), z 는 WeGo 틸트 TF 값 그대로(실측 필요).
-       이전 값: WeGo static TF (0.23, 0.05, 0.06), Webots (0.096, 0.015, 0.03) -->
-  <xacro:orbbec_dabai parent="base_link" name="camera" xyz="0.15 -0.005 0.06"
+  <!-- base_link → camera_link
+       real:   x·y 는 실물 실측(약 0.15, −0.005), z 는 WeGo 틸트 TF 값 그대로(실측 필요). 이전 값: WeGo static TF (0.23, 0.05, 0.06)
+       webots: Webots 모델의 깊이 렌즈 자리 (LimoFourDiff.proto 주석) -->
+  <xacro:property name="camera_xyz" value="${dict(real='0.15 -0.005 0.06', webots='0.096 0.015 0.03')['$(arg platform)']}"/>
+  <xacro:orbbec_dabai parent="base_link" name="camera" xyz="${camera_xyz}"
                       pitch="$(arg camera_pitch)" driver_tf="$(arg camera_driver_tf)"/>
 </robot>
